File: EAGLE/Volumetric Control Board.brd (EAGLE design)
At the start: 160 x 100 mm, 2 parts, among them U1 SN74LVC245AN

Commit message: EAGLE stuff started
Parts:
- removed U1: SN74LVC245AN, volumetric_display:SN74LVC245AN
- added U2: SN74HCT125NG4, volumetric_display:N14_TEX
Connections:
- removed net DIR3.3: U1.3
- removed net DIR5: U1.17
- removed net STEP3.3: U1.2
- removed net STEP5: U1.18
- new net DIR_5V: U2.6
- new net STEP_5V: U2.3
- net 5V: now also U2.10, U2.13, U2.14; no longer U1.1, U1.20
- net DIR: now also U2.5
- net GND: now also U2.1, U2.11, U2.12, U2.4, U2.7, U2.8, U2.9; no longer U1.10, U1.11, U1.12, U1.13, U1.14, U1.15, U1.16, U1.19, U1.4, U1.5, U1.6, U1.7, U1.8, U1.9
- net STEP: now also U2.2
Changed lines of the file:
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@@
 <?xml version="1.0" encoding="utf-8"?>
 <!DOCTYPE eagle SYSTEM "eagle.dtd">
-<eagle version="9.6.1">
+<eagle version="9.5.2">
 <drawing>
 <settings>
@@
 <elements>
 <element name="U$1" library="volumetric_display" library_urn="urn:adsk.eagle:library:31895123" package="TEENSY3.6" package3d_urn="urn:adsk.eagle:package:31895234/4" value="TEENSY3.6" x="-8.89" y="62.23" smashed="yes"/>
-<element name="U1" library="volumetric_display" library_urn="urn:adsk.eagle:library:31895123" package="SN74LVC245AN" package3d_urn="urn:adsk.eagle:package:31895306/3" value="SN74LVC245AN" x="-34.29" y="2.54" smashed="yes">
-<attribute name="COPYRIGHT" value="Copyright (C) 2021 Ultra Librarian. All rights reserved." x="-34.29" y="2.54" size="1.778" layer="27" display="off"/>
-<attribute name="DIGI-KEY_PART_NUMBER_1" value="296-8503-5-ND" x="-34.29" y="2.54" size="1.778" layer="27" display="off"/>
-<attribute name="DIGI-KEY_PART_NUMBER_2" value="2156-SN74LVC245AN-ND" x="-34.29" y="2.54" size="1.778" layer="27" display="off"/>
-<attribute name="MANUFACTURER_PART_NUMBER" value="SN74LVC245AN" x="-34.29" y="2.54" size="1.778" layer="27" display="off"/>
-<attribute name="MFR_NAME" value="Texas Instruments" x="-34.29" y="2.54" size="1.778" layer="27" display="off"/>
-<attribute name="NAME" x="-41.3766" y="13.335" size="1.27" layer="25" ratio="6" rot="SR0"/>
-<attribute name="VALUE" x="-39.8272" y="13.335" size="1.27" layer="27" ratio="6" rot="SR0"/>
+<element name="U2" library="volumetric_display" library_urn="urn:adsk.eagle:library:31895123" package="N14_TEX" package3d_urn="urn:adsk.eagle:package:31935452/2" value="SN74HCT125NG4" x="-52.07" y="17.78" smashed="yes">
+<attribute name="COPYRIGHT" value="Copyright (C) 2021 Ultra Librarian. All rights reserved." x="-52.07" y="17.78" size="1.778" layer="27" display="off"/>
+<attribute name="DIGI-KEY_PART_NUMBER_1" value="SN74HCT125NG4-ND" x="-52.07" y="17.78" size="1.778" layer="27" display="off"/>
+<attribute name="MANUFACTURER_PART_NUMBER" value="SN74HCT125NG4" x="-52.07" y="17.78" size="1.778" layer="27" display="off"/>
+<attribute name="MFR_NAME" value="Texas Instruments" x="-52.07" y="17.78" size="1.778" layer="27" display="off"/>
+<attribute name="NAME" x="-51.5366" y="9.525" size="1.27" layer="25" ratio="6" rot="SR0"/>
+<attribute name="VALUE" x="-49.9872" y="9.525" size="1.27" layer="27" ratio="6" rot="SR0"/>
 </element>
 </elements>
@@
 <contactref element="U$1" pad="GND_B"/>
 <contactref element="U$1" pad="GND"/>
-<contactref element="U1" pad="19"/>
-<contactref element="U1" pad="4"/>
-<contactref element="U1" pad="10"/>
-<contactref element="U1" pad="9"/>
-<contactref element="U1" pad="8"/>
-<contactref element="U1" pad="7"/>
-<contactref element="U1" pad="6"/>
-<contactref element="U1" pad="5"/>
-<contactref element="U1" pad="16"/>
-<contactref element="U1" pad="11"/>
-<contactref element="U1" pad="15"/>
-<contactref element="U1" pad="14"/>
-<contactref element="U1" pad="13"/>
-<contactref element="U1" pad="12"/>
-<wire x1="-8.89" y1="26.67" x2="-24.13" y2="62.23" width="0" layer="19" extent="1-1"/>
-<wire x1="-34.29" y1="22.86" x2="-8.89" y2="26.67" width="0" layer="19" extent="1-1"/>
-<wire x1="-34.29" y1="15.24" x2="-34.29" y2="22.86" width="0" layer="19" extent="1-1"/>
-<wire x1="-34.29" y1="12.7" x2="-34.29" y2="15.24" width="0" layer="19" extent="1-1"/>
-<wire x1="-34.29" y1="10.16" x2="-34.29" y2="12.7" width="0" layer="19" extent="1-1"/>
-<wire x1="-34.29" y1="7.62" x2="-34.29" y2="10.16" width="0" layer="19" extent="1-1"/>
-<wire x1="-34.29" y1="5.08" x2="-34.29" y2="7.62" width="0" layer="19" extent="1-1"/>
-<wire x1="-34.29" y1="2.54" x2="-34.29" y2="5.08" width="0" layer="19" extent="1-1"/>
-<wire x1="-41.91" y1="2.54" x2="-34.29" y2="2.54" width="0" layer="19" extent="1-1"/>
-<wire x1="-41.91" y1="5.08" x2="-41.91" y2="2.54" width="0" layer="19" extent="1-1"/>
-<wire x1="-41.91" y1="7.62" x2="-41.91" y2="5.08" width="0" layer="19" extent="1-1"/>
-<wire x1="-41.91" y1="10.16" x2="-41.91" y2="7.62" width="0" layer="19" extent="1-1"/>
-<wire x1="-41.91" y1="12.7" x2="-41.91" y2="10.16" width="0" layer="19" extent="1-1"/>
-<wire x1="-41.91" y1="15.24" x2="-41.91" y2="12.7" width="0" layer="19" extent="1-1"/>
-<wire x1="-41.91" y1="17.78" x2="-41.91" y2="15.24" width="0" layer="19" extent="1-1"/>
+<contactref element="U2" pad="7"/>
+<contactref element="U2" pad="1"/>
+<contactref element="U2" pad="4"/>
+<contactref element="U2" pad="12"/>
+<contactref element="U2" pad="11"/>
+<contactref element="U2" pad="9"/>
+<contactref element="U2" pad="8"/>
+<wire x1="-52.07" y1="10.16" x2="-52.07" y2="2.54" width="0" layer="19" extent="1-1"/>
+<wire x1="-44.45" y1="2.54" x2="-52.07" y2="2.54" width="0" layer="19" extent="1-1"/>
+<wire x1="-44.45" y1="5.08" x2="-44.45" y2="2.54" width="0" layer="19" extent="1-1"/>
+<wire x1="-44.45" y1="10.16" x2="-44.45" y2="5.08" width="0" layer="19" extent="1-1"/>
+<wire x1="-44.45" y1="12.7" x2="-44.45" y2="10.16" width="0" layer="19" extent="1-1"/>
+<wire x1="-52.07" y1="17.78" x2="-52.07" y2="10.16" width="0" layer="19" extent="1-1"/>
+<wire x1="-8.89" y1="26.67" x2="-44.45" y2="12.7" width="0" layer="19" extent="1-1"/>
+<wire x1="-24.13" y1="62.23" x2="-8.89" y2="26.67" width="0" layer="19" extent="1-1"/>
 </signal>
 <signal name="STEP">
 <contactref element="U$1" pad="2"/>
+<contactref element="U2" pad="2"/>
+<wire x1="-24.13" y1="54.61" x2="-52.07" y2="15.24" width="0" layer="19" extent="1-1"/>
 </signal>
 <signal name="DIR">
 <contactref element="U$1" pad="3"/>
+<contactref element="U2" pad="5"/>
+<wire x1="-24.13" y1="52.07" x2="-52.07" y2="7.62" width="0" layer="19" extent="1-1"/>
 </signal>
 <signal name="5V">
-<contactref element="U1" pad="20"/>
 <contactref element="U$1" pad="VIN"/>
-<contactref element="U1" pad="1"/>
-<wire x1="-34.29" y1="25.4" x2="-8.89" y2="62.23" width="0" layer="19" extent="1-1"/>
-<wire x1="-41.91" y1="25.4" x2="-34.29" y2="25.4" width="0" layer="19" extent="1-1"/>
-</signal>
-<signal name="DIR3.3">
-<contactref element="U1" pad="3"/>
-</signal>
-<signal name="STEP3.3">
-<contactref element="U1" pad="2"/>
-</signal>
-<signal name="STEP5">
-<contactref element="U1" pad="18"/>
-</signal>
-<signal name="DIR5">
-<contactref element="U1" pad="17"/>
+<contactref element="U2" pad="14"/>
+<contactref element="U2" pad="13"/>
+<contactref element="U2" pad="10"/>
+<wire x1="-44.45" y1="17.78" x2="-8.89" y2="62.23" width="0" layer="19" extent="1-1"/>
+<wire x1="-44.45" y1="15.24" x2="-44.45" y2="17.78" width="0" layer="19" extent="1-1"/>
+<wire x1="-44.45" y1="7.62" x2="-44.45" y2="15.24" width="0" layer="19" extent="1-1"/>
+</signal>
+<signal name="STEP_5V">
+<contactref element="U2" pad="3"/>
+</signal>
+<signal name="DIR_5V">
+<contactref element="U2" pad="6"/>
 </signal>
 </signals>

Commit message: adsf
Parts:
- added C1, C5: 10uF, rcl:C1206
- added C2, C6: 1uF, rcl:C1206
- added C3, C7: 0.1uF, rcl:C1206
- added C4, C8: 0.01uF, rcl:C1206
- added J1, J3: B6B-PH-K-S(LF)(SN), volumetric_display:CONN_B6B-PH-K-S_JST
- added J2: B8B-PH-K-S(LF)(SN), volumetric_display:JST_B8B-PH-K-S(LF)(SN)
- moved U2 59.5 mm to (7.37, 19.4), turned to 270 degrees
- moved U$1 58.3 mm to (-29.2, 7.62), turned to 90 degrees
Connections:
- new net 3.3V: C5.1, C6.1, C7.1, C8.1, J2.7, U$1.3.3V_A
- new net CS: J2.3, U$1.9
- new net D/C: J2.4, U$1.10
- new net MISO: J2.2, U$1.12
- new net MOSI: J2.1, U$1.11
- new net SCLK: J2.5, U$1.13
- new net USB_DM: J3.2, U$1.USB_DM
- new net USB_DP: J3.3, U$1.USB_DP
- net 5V: now also C1.1, C2.1, C3.1, C4.1, J3.1, U$1.USB_5V
- net DIR_5V: now also J1.3
- net GND: now also C1.2, C2.2, C3.2, C4.2, C5.2, C6.2, C7.2, C8.2, J1.4, J2.6, J3.4, U$1.USB_GND, U$1.USB_GND2
- net STEP_5V: now also J1.2
Routing:
- net 3.3V: track 0.00 -> 68.7 mm
- net STEP: track 0.00 -> 55.2 mm
- net 5V: track 0.00 -> 51.2 mm
- net DIR: track 0.00 -> 42.6 mm
- net USB_DP: track 0.00 -> 37.4 mm
- net USB_DM: track 0.00 -> 35.3 mm
- net DIR_5V: track 0.00 -> 30.6 mm
- net STEP_5V: track 0.00 -> 29.5 mm, vias 0 -> 1
- net SCLK: track 0.00 -> 27.3 mm
- net CS: track 0.00 -> 11.7 mm
- net MOSI: track 0.00 -> 11.3 mm
- net D/C: track 0.00 -> 9.82 mm
- net MISO: track 0.00 -> 9.36 mm
- added copper zone on layer 1, net 5V
- added copper zone on layer 1, net GND
- added copper zone on layer 16, net GND
Other:
- board size 160 x 100 mm -> 65 x 64.9 mm
- board text added: "OLED"
- board text added: "STEP/DIR"
- board text added: "USB"
- board text added: "VOLUMETRIC DISPLAY REV A"
