File: EAGLE/Volumetric Control Board.sch (EAGLE design)
At the start: 2 parts, among them U1 SN74LVC245AN

Commit message: EAGLE stuff started
Parts:
- removed U1: SN74LVC245AN, volumetric_display:SN74LVC245AN
- added U2: SN74HCT125NG4, volumetric_display:SN74HCT125NG4
Connections:
- removed net DIR3.3: U1.A2
- removed net DIR5: U1.B2
- removed net STEP3.3: U1.A1
- removed net STEP5: U1.B1
- new net DIR_5V: U2.2Y
- new net STEP_5V: U2.1Y
- net 5V: now also U2.!3OE, U2.!4OE, U2.VCC; no longer U1.DIR, U1.VCC
- net DIR: now also U2.2A
- net GND: now also U2.!1OE, U2.!2OE, U2.3A, U2.3Y, U2.4A, U2.4Y, U2.GND; no longer U1.!OE, U1.A3, U1.A4, U1.A5, U1.A6, U1.A7, U1.A8, U1.B3, U1.B4, U1.B5, U1.B6, U1.B7, U1.B8, U1.GND
- net STEP: now also U2.1A
Other:
- note removed: "NOPE. You need tri-state Buffer? SN54AHCT125"

Commit message: adsf
Parts:
- added C1, C5: 10uF, rcl:C-USC1206
- added C2, C6: 1uF, rcl:C-USC1206
- added C3, C7: 0.1uF, rcl:C-USC1206
- added C4, C8: 0.01uF, rcl:C-USC1206
- added J1, J3: B6B-PH-K-S(LF)(SN), volumetric_display:B6B-PH-K-S(LF)(SN)
- added J2: B8B-PH-K-S(LF)(SN), volumetric_display:B8B-PH-K-S(LF)(SN)
Connections:
- new net 3.3V: C5.1, C6.1, C7.1, C8.1, J2.P7, U$1.3.3V_A
- new net CS: J2.P3, U$1.9
- new net D/C: J2.P4, U$1.10
- new net MISO: J2.P2, U$1.12
- new net MOSI: J2.P1, U$1.11
- new net SCLK: J2.P5, U$1.13
- new net USB_DM: J3.2, U$1.USB_DM
- new net USB_DP: J3.3, U$1.USB_DP
- net 5V: now also C1.1, C2.1, C3.1, C4.1, J3.1, U$1.USB_5V
- net DIR_5V: now also J1.3
- net GND: now also C1.2, C2.2, C3.2, C4.2, C5.2, C6.2, C7.2, C8.2, J1.4, J2.P6, J3.4, U$1.USB_GND, U$1.USB_GND2
- net STEP_5V: now also J1.2
Other:
- note added: "OLED Connector"
- note added: "Slip ring Pair #1 USB"
- note added: "Slip ring Pair #2"
